File: Hardware/dspic33ch/dspic33ch-revc.brd (EAGLE design)
At the start: 85 x 65 mm, 32 parts, among them IC1 DSPIC33CH512MP208-I_PT, IC2 AP2114HA-3.3TRG1, J1 USB_MINI-B_SMT, Y1 DSC6083CI1A-350K000T

Commit message: revc final gerbers produced
Routing:
- net GND: track 412.7 -> 413.5 mm
Other:
- board size 85 x 65 mm -> 85 x 64 mm
